Commit message: Add odom-to-base_link TF and synthetic wheel joint state nodes

File: src/robot_description/urdf/ugv_beast.urdf (robot description, URDF)
Before this commit: robot ugv_beast, 13 links, 12 joints
Links:
- removed link pt_base_link
- removed link pt_camera_link
- removed link pt_link1
- removed link pt_link2
- link 3d_camera_link: mass 0.043316 -> None; geometry collision mesh filename=package://robot_description/meshes/3d_camera_link.stl; visual mesh filename=package://robot_description/meshes/3d_camera_link.stl
- link base_lidar_link: mass 0.0418000091653573 -> None; geometry collision mesh filename=package://robot_description/meshes/base_lidar_link.stl; visual mesh filename=package://robot_description/meshes/base_lidar_link.stl
- link base_link: mass 2.03227373732274 -> 2.032; geometry collision mesh filename=package://robot_description/meshes/base_link.stl; visual mesh filename=package://robot_description/meshes/base_link.stl
- link left_down_wheel_link: mass 0.00565722297095184 -> None; geometry collision mesh filename=package://robot_description/meshes/left_down_wheel_link.stl; visual mesh filename=package://robot_description/meshes/left_down_wheel_link.stl
- link left_up_wheel_link: mass 0.0602574557338752 -> None; geometry collision mesh filename=package://robot_description/meshes/left_up_wheel_link.stl; visual mesh filename=package://robot_description/meshes/left_up_wheel_link.stl
- link right_down_wheel_link: mass 0.00565722297095184 -> None; geometry collision mesh filename=package://robot_description/meshes/right_down_wheel_link.stl; visual mesh filename=package://robot_description/meshes/right_down_wheel_link.stl
- link right_up_wheel_link: mass 0.0602574557338752 -> None; geometry collision mesh filename=package://robot_description/meshes/right_up_wheel_link.stl; visual mesh filename=package://robot_description/meshes/right_up_wheel_link.stl
Joints:
- removed joint pt_base_link_joint
- removed joint pt_base_link_to_pt_link1
- removed joint pt_link1_to_pt_link2
- removed joint pt_link2_to_pt_camera_link
- joint 3d_camera_link_joint: axis 0 0 0 -> (none); origin xyz=0.069874862129561 0 0.0792560807319928 rpy=0 0 0 -> xyz=0.0699 0 0.0793 rpy=0 0 0
- joint base_joint: origin xyz=0.000460087791654118 6.50856019576702E-10 0.08 rpy=0 0 0 -> xyz=0 0 0.08 rpy=0 0 0
- joint base_lidar_link_joint: axis 0 0 0 -> (none); origin xyz=0.0443794126815426 0 0.0973030807319928 rpy=0 0 1.5708 -> xyz=0.0444 0 0.0973 rpy=0 0 1.5708
- joint left_down_wheel_link_joint: origin xyz=-0.0722382907996229 0.0707110003635451 0.0356492872743132 rpy=0 0 0 -> xyz=-0.0722 0.0707 0.0356 rpy=0 0 0
- joint left_up_wheel_link_joint: origin xyz=0.0832175533230826 0.0619109945296507 0.0261492872743138 rpy=0 0 0 -> xyz=0.0832 0.0619 0.0261 rpy=0 0 0
- joint right_down_wheel_link_joint: origin xyz=-0.0722382907996239 -0.0707110003635441 0.0356492872743132 rpy=0 0 0 -> xyz=-0.0722 -0.0707 0.0356 rpy=0 0 0
- joint right_up_wheel_link_joint: origin xyz=0.0832175533230817 -0.0619109945296519 0.0261492872743138 rpy=0 0 0 -> xyz=0.0832 -0.0619 0.0261 rpy=0 0 0

Commit message: Added teleop_twist_keyboard as a submodule

File: src/robot_description/urdf/ugv_beast.urdf (robot description, URDF)
Before this commit: robot ugv_beast, 9 links, 8 joints
Links:
- removed link 3d_camera_link
- added link camera0_link, mass 0.043316; collision mesh filename=package://robot_description/meshes/3d_camera_link.stl; visual mesh filename=package://robot_description/meshes/3d_camera_link.stl
- link base_lidar_link: mass None -> 0.0418000091653573
- link base_link: mass 2.032 -> 2.03227373732274
- link left_down_wheel_link: mass None -> 0.00565722297095184
- link left_up_wheel_link: mass None -> 0.0602574557338752
- link right_down_wheel_link: mass None -> 0.00565722297095184
- link right_up_wheel_link: mass None -> 0.0602574557338752
Joints:
- removed joint 3d_camera_link_joint
- added joint camera0_link_joint: type fixed, parent base_link, child camera0_link, origin xyz=0.07 0 0.055 rpy=0 0 0
- joint base_joint: origin xyz=0 0 0.08 rpy=0 0 0 -> xyz=0 0 0.09 rpy=0 0 0
- joint base_lidar_link_joint: origin xyz=0.0444 0 0.0973 rpy=0 0 1.5708 -> xyz=0.0443794126815426 0 0.0973030807319928 rpy=0 0 1.5708
- joint left_down_wheel_link_joint: origin xyz=-0.0722 0.0707 0.0356 rpy=0 0 0 -> xyz=-0.0722382907996229 0.0707110003635451 0.0356492872743132 rpy=0 0 0
- joint left_up_wheel_link_joint: origin xyz=0.0832 0.0619 0.0261 rpy=0 0 0 -> xyz=0.0832175533230826 0.0619109945296507 0.0261492872743138 rpy=0 0 0
- joint right_down_wheel_link_joint: origin xyz=-0.0722 -0.0707 0.0356 rpy=0 0 0 -> xyz=-0.0722382907996239 -0.0707110003635441 0.0356492872743132 rpy=0 0 0
- joint right_up_wheel_link_joint: origin xyz=0.0832 -0.0619 0.0261 rpy=0 0 0 -> xyz=0.0832175533230817 -0.0619109945296519 0.0261492872743138 rpy=0 0 0
